File: electronics/kicad/rockobot/rockobot.kicad_sch (KiCad schematic)
At the start: 33 parts

Commit message: Updated schematic with pin info about L298N driver
Other:
- note added: "In order (D3 to D9 except D8): ENA, IN1 to IN4, ENB"
- note added: "Pins 3 and 9 are PWM-able, that is why they are used for ENA and ENB"
- note removed: "Pins 5 and 6 are PWM-able, that is why they are used for ENA and ENB"
Changed lines of the file:
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@@
     (stroke (width 0) (type default))
   )
-  (text "Pins 5 and 6 are PWM-able, that is \nwhy they are used for ENA and ENB\n"
-    (at 78.74 105.41 0)
+  (text "Pins 3 and 9 are PWM-able, that is \nwhy they are used for ENA and ENB\n"
+    (at 92.71 78.74 0)
     (effects (font (size 0.85 0.85) bold) (justify left bottom))
   )
@@
     (at 62.23 152.4 0)
     (effects (font (size 1.27 1.27)) (justify left bottom))
+  )
+  (text "In order (D3 to D9 except D8):\nENA,\nIN1 to IN4,\nENB"
+    (at 88.9 95.25 0)
+    (effects (font (size 1.1 1.1)) (justify left bottom))
   )
   (symbol (lib_id "Connector:Conn_01x02_Socket") (at 73.66 33.02 270) (mirror x) (unit 1)
@@
   )
   (symbol (lib_id "Connector:Conn_01x06_Socket") (at 119.38 95.25 180) (unit 1)
-    (in_bom yes) (on_board yes) (dnp no) (fields_autoplaced)
-    (property "Reference" "Motor_Control1" (at 120.015 83.82 0)
+    (in_bom yes) (on_board yes) (dnp no)
+    (property "Reference" "Motor_Control1" (at 105.41 82.55 0)
       (effects (font (size 1.27 1.27)))
     )
-    (property "Value" "Conn_01x06_Socket" (at 120.015 86.36 0)
+    (property "Value" "Conn_01x06_Socket" (at 106.045 85.09 0)
       (effects (font (size 1.27 1.27)))
     )

Commit message: Fixed comment in schematic
Other:
- note added: "In order (D3 to D9 except D8): ENB, IN1 to IN4, ENA"
- note removed: "In order (D3 to D9 except D8): ENA, IN1 to IN4, ENB"
Changed lines of the file:
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@@
     (effects (font (size 1.27 1.27)) (justify left bottom))
   )
-  (text "In order (D3 to D9 except D8):\nENA,\nIN1 to IN4,\nENB"
+  (text "In order (D3 to D9 except D8):\nENB,\nIN1 to IN4,\nENA"
     (at 88.9 95.25 0)
     (effects (font (size 1.1 1.1)) (justify left bottom))
